File: solder.kicad_pcb (KiCad board)
At the start: 2 copper layers, 60 x 61 mm, 13 parts, among them M1 Motor_DC, SW2 SW_Push

Commit message: updated silkscreens
Parts:
- added G***: LOGO, LOGO, F.Cu at (134.5, 112.0)
- added G***: LOGO, LOGO, B.Cu at (144.0, 115.0)
- M1: moved to B.Cu
- moved M1 8.02 mm to (156.5, 97.5)
- moved SW2 0.35 mm to (146.8, 103.2)
Routing:
- net Net-(BT1-+): track 120.0 -> 107.9 mm
- net Net-(M1--): track 30.1 -> 32.9 mm
- net Net-(M1-+): track 13.0 -> 14.4 mm
